Commit message: update visual mesh

File: assets/allegro/allegro_internal.urdf (robot description, URDF)
Before this commit: robot allegro_hand_right, 21 links, 20 joints
Links:
- link link_11.0_tip: geometry collision sphere radius=0.01235; visual mesh filename=allegro/meshes/allegro/digitv2.obj
- link link_15.0_tip: geometry collision sphere radius=0.01235; visual mesh filename=allegro/meshes/allegro/digitv2.obj
- link link_3.0_tip: geometry collision sphere radius=0.01235; visual mesh filename=allegro/meshes/allegro/digitv2.obj
- link link_7.0_tip: geometry collision sphere radius=0.01235; visual mesh filename=allegro/meshes/allegro/digitv2.obj
